File: Block Schematic Munin 400/Block Schematic Munin 400.kicad_sch (KiCad schematic)
At the start: 11 parts

Commit message: Updated
Connections:
- net GND: no longer U?. (GND)
- net at U?. (TX): now also PA?. (PTT), U?. (GND)
- net at U?. (GND): now also U?.5
- net at PA?. (PTT): no longer U?. (GND)
- net at U?. (TX): now also LPF?. (RF_OUT)
- net at U?. (TRX): now also PA?. (PTT); no longer U?. (TX)
- net at LPF?. (RF_OUT): now also PA?. (PTT); no longer U?. (TX)
- new net: PA?. (PTT), U?. (GND), U?. (TX)
- new net: U?. (GND), U?. (GND), U?. (GND) (x2)
- new net: PA?. (PTT), U?. (GND) (x2)
- new net: U?. (TRX), U?. (TX)
- now unconnected: PA?. (PTT), PA?. (PTT), PA?. (PTT), PA?. (PTT), PA?. (PTT), U?. (GND), U?. (GND)
Changed lines of the file:
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@@
-(kicad_sch (version 20210126) (generator eeschema)
+(kicad_sch (version 20210621) (generator eeschema)
   (paper "A4")
   (title_block
@@
     (stroke (width 0) (type solid) (color 0 0 0 0))
   )
-  (wire (pts (xy 16.51 144.78) (xy 28.575 144.78))
-    (stroke (width 0) (type solid) (color 0 0 0 0))
-  )
   (wire (pts (xy 18.415 38.735) (xy 18.415 40.005))
     (stroke (width 0) (type solid) (color 0 0 0 0))
   )
+  (wire (pts (xy 19.05 177.8) (xy 48.006 177.8))
+    (stroke (width 0) (type solid) (color 0 0 0 0))
+  )
   (wire (pts (xy 19.685 38.1) (xy 15.875 38.1))
     (stroke (width 0) (type solid) (color 0 0 0 0))
@@
     (stroke (width 0) (type solid) (color 0 0 0 0))
   )
-  (wire (pts (xy 28.575 143.51) (xy 28.575 144.78))
+  (wire (pts (xy 28.702 143.51) (xy 28.702 145.288))
+    (stroke (width 0) (type solid) (color 0 0 0 0))
+  )
+  (wire (pts (xy 28.702 145.288) (xy 37.592 145.288))
     (stroke (width 0) (type solid) (color 0 0 0 0))
   )
@@
     (stroke (width 0) (type solid) (color 0 0 0 0))
   )
-  (wire (pts (xy 30.48 143.51) (xy 30.48 145.415))
+  (wire (pts (xy 30.48 143.51) (xy 48.006 143.51))
     (stroke (width 0) (type solid) (color 0 0 0 0))
   )
@@
     (stroke (width 0) (type solid) (color 0 0 0 0))
   )
-  (wire (pts (xy 37.465 145.415) (xy 30.48 145.415))
-    (stroke (width 0) (type solid) (color 0 0 0 0))
-  )
   (wire (pts (xy 37.465 147.32) (xy 37.465 145.415))
     (stroke (width 0) (type solid) (color 0 0 0 0))
@@
     (stroke (width 0) (type solid) (color 0 0 0 0))
   )
+  (wire (pts (xy 48.006 177.8) (xy 48.006 143.51))
+    (stroke (width 0) (type solid) (color 0 0 0 0))
+  )
   (wire (pts (xy 48.895 67.31) (xy 48.895 73.66))
     (stroke (width 0) (type solid) (color 0 0 0 0))
@@
     (stroke (width 0) (type solid) (color 0 0 0 0))
   )
+  (wire (pts (xy 194.8 89.1) (xy 194.8 89.4))
+    (stroke (width 0) (type solid) (color 0 0 0 0))
+  )
   (wire (pts (xy 194.945 71.12) (xy 204.47 71.12))
     (stroke (width 0) (type solid) (color 0 0 0 0))
@@
     (stroke (width 0) (type solid) (color 0 0 0 0))
   )
+  (wire (pts (xy 195 86.9) (xy 195 87))
+    (stroke (width 0) (type solid) (color 0 0 0 0))
+  )
+  (wire (pts (xy 195 86.9) (xy 203.8 86.9))
+    (stroke (width 0) (type solid) (color 0 0 0 0))
+  )
   (wire (pts (xy 202.565 38.1) (xy 202.565 39.37))
     (stroke (width 0) (type solid) (color 0 0 0 0))
@@
     (stroke (width 0) (type solid) (color 0 0 0 0))
   )
+  (wire (pts (xy 203.8 89.4) (xy 194.8 89.4))
+    (stroke (width 0) (type solid) (color 0 0 0 0))
+  )
   (wire (pts (xy 204.47 39.37) (xy 202.565 39.37))
     (stroke (width 0) (type solid) (color 0 0 0 0))
@@
   (text "12+10m" (at 218.44 121.92 180)
     (effects (font (size 1.27 1.27)) (justify right bottom))
-  )
-  (symbol (lib_id "power:GND") (at 16.51 144.78 0) (unit 1)
-    (in_bom yes) (on_board yes)
-    (property "Reference" "#PWR?" (id 0) (at 16.51 151.13 0)
-      (effects (font (size 1.27 1.27)) hide)
-    )
-    (property "Value" "GND" (id 1) (at 16.51 149.1044 0))
-    (property "Footprint" "" (id 2) (at 16.51 144.78 0)
-      (effects (font (size 1.27 1.27)) hide)
-    )
-    (property "Datasheet" "" (id 3) (at 16.51 144.78 0)
-      (effects (font (size 1.27 1.27)) hide)
-    )
-    (pin "1")
   )
   (symbol (lib_id "power:GND") (at 33.02 95.25 0) (unit 1)
@@
     (pin "")
     (pin "")
+    (pin "10")
+    (pin "9")
   )
   (symbol (lib_id "KjellKarlsen:PA_Protection_Board") (at 97.79 102.235 0) (unit 1)
@@
   )
   (symbol_instances
-    (path "/05523b60-853e-4f1d-a30a-da52a5702edd"
-      (reference "#PWR?") (unit 1) (value "GND") (footprint "")
-    )
     (path "/3a1f40f0-105f-458d-8999-7e3a34fb490d"
       (reference "#PWR?") (unit 1) (value "GND") (footprint "")
